File: v0.1/hardware/sweet-p.kicad_pcb (KiCad board)
At the start: 2 copper layers, 83 x 73 mm, 43 parts, among them J1 Screw_Terminal_01x03, J10 Micro_SD_Card, J2 Screw_Terminal_01x02, J3 Conn_01x04_Female, J5 Screw_Terminal_01x05, J6 Conn_01x02_Socket, J7 Conn_01x06_Pin, J8 Conn_01x08_Socket, SW1 SW_Push, U1 adafruit_tpl511x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

Commit message: update
Parts:
- removed S2: EG1218, digikey-footprints:Switch_Slide_11.6x4mm_EG1218
- removed U2: MCP1700x-120xxTO, Package_TO_SOT_THT:TO-92_Inline
- removed U4: ssd1306, footprints:ssd1306_a
- removed U7: ds3231, footprints:ds3231_adafruit_breakout
- removed U8: P78A05-1000, footprints:CONV_P78A05-1000
- added J4: Conn_01x04_Socket, Connector_PinHeader_2.54mm:PinHeader_1x04_P2.54mm_Vertical, F.Cu at (66.0, 17.0)
- added J9: Conn_01x08_Socket, Connector_PinHeader_2.54mm:PinHeader_1x08_P2.54mm_Vertical, F.Cu at (21.0, 43.5)
- added JP1: Jumper_2_Open, Jumper:SolderJumper-2_P1.3mm_Open_Pad1.0x1.5mm, B.Cu at (74.0, 47.1)
- J10: value Micro_SD_Card -> Conn_01x04_Socket; footprint footprints:DM3D-SF_outline -> footprints:ssd1306_a
- J5: value Screw_Terminal_01x05 -> Conn_01x06_Socket; footprint TerminalBlock_Phoenix:TerminalBlock_Phoenix_MKDS-1,5-5-5.08_1x05_P5.08mm_Horizontal -> Connector_PinHeader_2.54mm:PinHeader_1x06_P2.54mm_Vertical
- J7: value Conn_01x06_Pin -> Screw_Terminal_01x04; footprint Connector_PinHeader_2.54mm:PinHeader_1x06_P2.54mm_Vertical -> TerminalBlock_Phoenix:TerminalBlock_Phoenix_MKDS-1,5-4_1x04_P5.00mm_Horizontal
- J8: value Conn_01x08_Socket -> Conn_01x04_Socket; footprint Connector_PinSocket_2.54mm:PinSocket_1x08_P2.54mm_Vertical -> Connector_PinHeader_2.54mm:PinHeader_1x04_P2.54mm_Vertical
- moved U3 138.9 mm to (57.0, 2.55)
- moved H3 107.9 mm to (0.00, 0.00)
- moved H4 107.1 mm to (0.00, 70.0)
- moved R3 86.1 mm to (73.1, 2.75), turned to 0 degrees
- moved R4 83.6 mm to (69.2, 2.75), turned to 0 degrees
- moved SW1 81.5 mm to (84.0, 0.00), turned to 0 degrees
- moved J10 77.9 mm to (91.8, 10.5)
- moved H1 75.3 mm to (100.0, 0.00)
- moved H2 74.0 mm to (100.0, 70.0)
- moved J8 63.0 mm to (43.5, 48.1), turned to 0 degrees
- moved J6 53.2 mm to (101.8, 46.0), turned to 0 degrees
- moved R1 49.0 mm to (95.8, 47.6), turned to -90 degrees
- moved C2 47.6 mm to (5.75, 42.0), turned to 0 degrees
- moved D1 47.2 mm to (5.96, 35.5), turned to 0 degrees
- moved R2 46.3 mm to (95.8, 43.8), turned to -90 degrees
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Connections:
- net ONEWIRE_11 renamed ONEWIRE
- A2 pad 10: A5 -> BUTTON
- A2 pad 14: RX_D2 -> D2
- A2 pad 15: RX -> MESH_RX
- A2 pad 16: TX -> MESH_TX
- A2 pad 21: SAT_EN -> D9
- A2 pad 22: SD_CS -> DEPTH_PULL
- A2 pad 28: 5V_TIMER -> V_TIMER
- A2 pad 6: BATT_A1 -> A1
- A2 pad 8: A3 -> DEPTH_TX
- A2 pad 9: TX_A4 -> BATT_MEASURE
- C2 pad 1: 5V_TIMER -> V_TIMER
- J10 pad 1: unconnected-(J10-DAT2-Pad1) -> +3V3
- J10 pad 2: SD_CS -> GND
- J10 pad 3: MOSI -> SCL
- J10 pad 4: +3V3 -> SDA
- J2 pad 1: VEXT -> MESH_BAT
- J5 pad 1: GND -> A0
- J5 pad 2: +3V3 -> A1
- J5 pad 3: RX_D2 -> A2
- J5 pad 4: TX_A4 -> DEPTH_TX
- J5 pad 5: D12 -> BUTTON
- J7 pad 2: 5V_DC -> DEPTH_TX
- J7 pad 3: SAT_EN -> DEPTH_PULL
- J7 pad 4: TX -> GND
- J8 pad 1: GND -> +3V3
- J8 pad 2: +3V3 -> SCL
- J8 pad 3: 5V_TIMER -> SDA
- J8 pad 4: SDA -> GND
- R13 pad 1: VEXT -> MESH_BAT
- R13 pad 2: BATT_A1 -> BATT_MEASURE
- R14 pad 1: VEXT -> MESH_BAT
- R14 pad 2: BATT_A1 -> BATT_MEASURE
- R15 pad 1: BATT_A1 -> BATT_MEASURE
- R16 pad 1: BATT_A1 -> BATT_MEASURE
- R17 pad 1: SAT_EN -> DEPTH_PULL
- R18 pad 1: SAT_EN -> DEPTH_PULL
- R3 pad 2: A5 -> BUTTON
- R4 pad 2: A5 -> BUTTON
- SW1 pad 1: A5 -> BUTTON
- U1 pad 1: 5V_DC -> MESH_BAT
- U1 pad 4: 5V_TIMER -> V_TIMER
- U3 pad 1: unconnected-(U3-BAT-Pad1) -> BAT
- U3 pad 2: unconnected-(U3-IO2-Pad2) -> IO2
- U3 pad 3: unconnected-(U3-IO1-Pad3) -> IO1
- U3 pad 4: unconnected-(U3-AIN1-Pad4) -> AIN1
- U3 pad 5: unconnected-(U3-RX1-Pad5) -> MESH_TX
- U3 pad 6: unconnected-(U3-TX1-Pad6) -> MESH_RX
- U3 pad 7: unconnected-(U3-GND-Pad7) -> GND
Other:
- board size 83 x 73 mm -> 108 x 77 mm
- board text added: "3V3"
- board text added: "A1"
- board text added: "AIN1"
- board text added: "B0"
- board text added: "BAT"
- board text added: "BTN"
- board text added: "D2"
- board text added: "D9"
- board text added: "DP_4"
- board text added: "DP_5"
- board text added: "DTX"
- board text added: "IO1"
- board text added: "IO2"
- board text added: "ITSY-BITSY"
- board text added: "MESH_RX"
- board text added: "MESH_TX"
- board text added: "RAK4631 + RAK19007"
- board text added: "RX1"
- board text added: "TX1"
- board text added: "V_TIMER"
- board text removed: "5V"
- board text removed: "5VT"
- board text removed: "A3"
- board text removed: "FORCE SEND"
- board text removed: "OFF"
- board text removed: "ON"
- board text removed: "RX"
- board text removed: "RX2"
- board text removed: "SEN"
- board text removed: "TX"
- board text removed: "TX2"
- board text removed: "VEXT"
- board text removed: "github.com/edgecollective/sweet-p"
- board text removed: "itsybitsy"
- board text removed: "p78a05-1000"
- board text removed: "ssd1306"
- board text removed: "sweet-p ver 0.4a"

Commit message: update
Parts:
- moved J7 15.0 mm to (76.8, 65.2), turned to 0 degrees
- moved J10 0.44 mm to (91.3, 10.5)
Connections:
- J7 pad 1: +3V3 -> GND
- J7 pad 2: DEPTH_TX -> +3V3
- J7 pad 3: DEPTH_PULL -> DEPTH_TX
- J7 pad 4: GND -> DEPTH_PULL
Other:
- board size 108 x 77 mm -> 107.5 x 77 mm
