File: v0.1/hardware/sweet-p.kicad_sch (KiCad schematic)
At the start: 38 parts, among them J1 Screw_Terminal_01x03, J2 Screw_Terminal_01x02, J3 Conn_01x04_Female, J5 Conn_01x06_Socket, J6 Conn_01x02_Socket, J7 Screw_Terminal_01x04, J9 Conn_01x08_Socket, SW1 SW_Push, U1 adafruit_tpl511x, U4 ssd1306

Commit message: update
Parts:
- removed U4: ssd1306, footprints:ssd1306_a, symbol picoco2:ssd1306
- added J10: Conn_01x04_Socket, footprints:ssd1306_b, symbol Connector:Conn_01x04_Socket
- added J4, J8: Conn_01x04_Socket, Connector_PinHeader_2.54mm:PinHeader_1x04_P2.54mm_Vertical, symbol Connector:Conn_01x04_Socket
- added JP1: Jumper_2_Open, Jumper:SolderJumper-2_P1.3mm_Open_Pad1.0x1.5mm, symbol Jumper:Jumper_2_Open
- J5: footprint (none) -> Connector_PinHeader_2.54mm:PinHeader_1x06_P2.54mm_Vertical
- J7: footprint (none) -> TerminalBlock_Phoenix:TerminalBlock_Phoenix_MKDS-1,5-4_1x04_P5.00mm_Horizontal
- J9: footprint (none) -> Connector_PinHeader_2.54mm:PinHeader_1x08_P2.54mm_Vertical
Connections:
- net VEXT is gone; now on net MESH_BAT: R13.1, R14.1
- net +3V3: now also J7.1 (Pin_1), J10.1 (Pin_1), J8.1 (Pin_1); no longer J7.2 (Pin_2)
- net AIN1: now also J4.3 (Pin_3)
- net DEPTH_PULL: now also J7.3 (Pin_3); no longer J7.4 (Pin_4)
- net GND: now also J7.4 (Pin_4), J9.8 (Pin_8), J10.2 (Pin_2), J4.4 (Pin_4), J8.4 (Pin_4); no longer J7.1 (Pin_1)
- net IO2: now also J4.1 (Pin_1)
- net MESH_BAT: now also JP1.1 (A)
- net SCL: now also J10.3 (Pin_3), J8.2 (Pin_2)
- net SDA: now also J10.4 (Pin_4), J8.3 (Pin_3)
- net V_TIMER: now also JP1.2 (B)
- net DEPTH_RX renamed DEPTH_TX
- net DEPTH_TX: now also J7.2 (Pin_2); no longer J7.3 (Pin_3)
- net IO3 renamed IO1
- net IO1: now also J4.2 (Pin_2)
- no-connect marks 0 -> 1
Other:
- note added: "bypass_timer"

Commit message: update
Parts:
- J10: footprint footprints:ssd1306_b -> footprints:ssd1306_a
Connections:
- net +3V3: now also J7.2 (Pin_2); no longer J7.1 (Pin_1)
- net DEPTH_PULL: now also J7.4 (Pin_4); no longer J7.3 (Pin_3)
- net DEPTH_TX: now also J7.3 (Pin_3); no longer J7.2 (Pin_2)
- net GND: now also J7.1 (Pin_1); no longer J7.4 (Pin_4)
Changed lines of the file:
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@@
 	(wire
 		(pts
+			(xy 292.1 33.02) (xy 302.26 33.02)
+		)
+		(stroke
+			(width 0)
+			(type default)
+		)
+	)
+	(wire
+		(pts
 			(xy 133.35 118.11) (xy 142.24 118.11)
 		)
@@
 	(wire
 		(pts
+			(xy 284.48 30.48) (xy 302.26 30.48)
+		)
+		(stroke
+			(width 0)
+			(type default)
+		)
+	)
+	(wire
+		(pts
 			(xy 31.75 95.25) (xy 38.1 95.25)
 		)
@@
 	(global_label "DEPTH_TX"
 		(shape input)
-		(at 302.26 33.02 180)
+		(at 302.26 35.56 180)
 		(fields_autoplaced yes)
 		(effects
@@
 		)
 		(property "Intersheetrefs" "${INTERSHEET_REFS}"
-			(at 290.143 33.02 0)
+			(at 290.143 35.56 0)
 			(effects
 				(font
@@
 	(global_label "DEPTH_PULL"
 		(shape input)
-		(at 302.26 35.56 180)
+		(at 302.26 38.1 180)
 		(fields_autoplaced yes)
 		(effects
@@
 		)
 		(property "Intersheetrefs" "${INTERSHEET_REFS}"
-			(at 287.6634 35.56 0)
+			(at 287.6634 38.1 0)
 			(effects
 				(font
@@
 	(symbol
 		(lib_id "power:+3V3")
-		(at 302.26 30.48 0)
+		(at 292.1 33.02 0)
 		(unit 1)
 		(exclude_from_sim no)
@@
 		(fields_autoplaced yes)
 		(property "Reference" "#PWR030"
-			(at 302.26 34.29 0)
+			(at 292.1 36.83 0)
 			(effects
 				(font
@@
 		)
 		(property "Value" "+3V3"
-			(at 302.26 25.4 0)
+			(at 292.1 27.94 0)
 			(effects
 				(font
@@
 		)
 		(property "Footprint" ""
-			(at 302.26 30.48 0)
+			(at 292.1 33.02 0)
 			(effects
 				(font
@@
 		)
 		(property "Datasheet" ""
-			(at 302.26 30.48 0)
+			(at 292.1 33.02 0)
 			(effects
 				(font
@@
 		)
 		(property "Description" ""
-			(at 302.26 30.48 0)
+			(at 292.1 33.02 0)
 			(effects
 				(font
@@
 			)
 		)
-		(property "Footprint" "footprints:ssd1306_b"
+		(property "Footprint" "footprints:ssd1306_a"
 			(at 214.63 24.13 0)
 			(effects
@@
 		(lib_name "GND_11")
 		(lib_id "power:GND")
-		(at 302.26 38.1 0)
+		(at 284.48 30.48 0)
 		(unit 1)
 		(exclude_from_sim no)
@@
 		(fields_autoplaced yes)
 		(property "Reference" "#PWR029"
-			(at 302.26 44.45 0)
+			(at 284.48 36.83 0)
 			(effects
 				(font
@@
 		)
 		(property "Value" "GND"
-			(at 302.26 43.18 0)
+			(at 284.48 35.56 0)
 			(effects
 				(font
@@
 		)
 		(property "Footprint" ""
-			(at 302.26 38.1 0)
+			(at 284.48 30.48 0)
 			(effects
 				(font
@@
 		)
 		(property "Datasheet" ""
-			(at 302.26 38.1 0)
+			(at 284.48 30.48 0)
 			(effects
 				(font
@@
 		)
 		(property "Description" ""
-			(at 302.26 38.1 0)
+			(at 284.48 30.48 0)
 			(effects
 				(font
