File: remote/v0.2/hardware/mesh-depth/mesh-depth.kicad_pcb (KiCad board)
At the start: 2 copper layers, 107.5 x 77 mm, 42 parts, among them J1 Screw_Terminal_01x03, J10 Conn_01x04_Socket, J2 Screw_Terminal_01x02, J3 Conn_01x04_Female, J4 Conn_01x04_Socket, J5 Conn_01x06_Socket, J6 Conn_01x02_Socket, J7 Screw_Terminal_01x04, J8 Conn_01x04_Socket, J9 Conn_01x08_Socket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

Commit message: update
Other:
- board text added: "V_timer"
- board text added: "mesh_bat"
Changed lines of the file:
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@@
 		(layer "Edge.Cuts")
+	)
+	(gr_text "V_timer"
+		(at 74.5 36.4 90)
+		(layer "B.SilkS")
+		(effects
+			(font
+				(size 1.5 1.5)
+				(thickness 0.3)
+				(bold yes)
+			)
+			(justify left bottom mirror)
+		)
+	)
+	(gr_text "mesh_bat"
+		(at 74.6 48.9 90)
+		(layer "B.SilkS")
+		(effects
+			(font
+				(size 1.5 1.5)
+				(thickness 0.3)
+				(bold yes)
+			)
+			(justify left bottom mirror)
+		)
 	)
 	(gr_text "1W"
